Commit message: fixing urdf

File: src/vehicle_drivers/gem_description/urdf/e4/gem_e4.urdf.xacro (robot description, xacro)
@@ -583,4 +583,7 @@
   </joint>
   <!-- ************************************* Sensor Links ************************************* -->
+  <xacro:OS1_64 parent="top_rack_link" name="os_sensor" topic_points="/ouster/points" topic_imu ="/ouster/imu" hz="10" lasers="64" samples="512" min_range="0.9" max_range="75.0" noise="0.008" min_angle="-${M_PI}" max_angle="${M_PI}" lidar_link="os_lidar" imu_link="os_imu" vfov_min="-.26" vfov_max=".26" >
+    <origin xyz="0.02 0.42 0" rpy="1.5708 0 3.1416" />
+  </xacro:OS1_64>
   <link name="gps_antenna_main_link">
     <inertial>
@@ -706,4 +709,39 @@
     <child link="front_camera_link" />
     <axis xyz="0 0 0" />
+  </joint>
+  <link name="front_single_camera_link">
+    <collision>
+      <origin xyz="0 0 0" rpy="0 0 0"/>
+      <geometry>
+        <box size="0.05 0.05 0.05"/>
+      </geometry>
+    </collision>
+    <visual>
+      <origin xyz="0 0 0" rpy="0 0 0"/>
+      <geometry>
+        <box size="0.05 0.05 0.05"/>
+      </geometry>
+      <material name="red"/>
+    </visual>
+    <inertial>
+      <mass value="1e-5" />
+      <origin xyz="0 0 0" rpy="0 0 0"/>
+      <inertia ixx="1e-6" ixy="0" ixz="0" iyy="1e-6" iyz="0" izz="1e-6" />
+    </inertial>
+  </link>
+  <gazebo reference="front_single_camera_link">
+    <material>Gazebo/White</material>
+  </gazebo>
+  <!--
+  <joint name="gem_front_camera_joint" type="fixed">
+    <origin xyz="-0.045 0 0" rpy="-1.5708 3.1416 0"/>
+    <parent link="front_camera_link"/>
+    <child link="front_single_camera_link"/>
+  </joint>
+  -->
+  <joint name="gem_front_camera_joint" type="fixed">
+    <origin xyz="0 0 0" rpy="0 -1.57 0"/>
+    <parent link="front_camera_link"/>
+    <child link="front_single_camera_link"/>
   </joint>
   <link name="front_lidar_link">
@@ -805,4 +843,224 @@
     <parent link="imu_link"/>
     <child link="vsm"/>
+  </joint>
+   <!-- ************************* Corner Cameras ************************* -->
+  <!-- Front Left Corner Camera -->
+  <link name="front_left_corner_camera_link">
+    <!-- <collision>
+      <origin xyz="0 0 0" rpy="0 0 0"/>
+      <geometry>
+        <box size="0.02 0.02 0.01"/>
+      </geometry>
+    </collision> -->
+    <visual>
+      <origin xyz="0 0 0" rpy="0 0 0"/>
+      <geometry>
+        <box size="0.02 0.02 0.01"/>
+      </geometry>
+      <material name="red"/>
+    </visual>
+    <inertial>
+      <mass value="1e-5" />
+      <origin xyz="0 0 0" rpy="0 0 0"/>
+      <inertia ixx="1e-6" ixy="0" ixz="0" iyy="1e-6" iyz="0" izz="1e-6" />
+    </inertial>
+  </link>
+  <gazebo reference="front_left_corner_camera_link">
+    <material>Gazebo/Red</material>
+  </gazebo>
+  <joint name="front_left_corner_camera_joint" type="fixed">
+    <origin xyz="0.5 0.6545 1.75" rpy="0 0.785 0.785"/>
+    <parent link="base_link"/>
+    <child link="front_left_corner_camera_link"/>
+    <axis xyz="0 0 0" />
+  </joint>
+  <!-- Front Left Corner Camera Optical Frame (For ROS Image/CameraInfo messages) -->
+  <link name="front_left_corner_camera_optical_frame"/>
+  <joint name="front_left_corner_camera_optical_joint" type="fixed">
+    <!-- -90 deg Roll, -90 deg Yaw rotation to align body frame with optical frame -->
+    <origin xyz="0 0 0" rpy="-1.5707963 0 -1.5707963"/>
+    <parent link="front_left_corner_camera_link"/>
+    <child link="front_left_corner_camera_optical_frame"/>
+  </joint>
+  <!-- Front Right Corner Camera -->
+  <link name="front_right_corner_camera_link">
+    <!-- <collision>
+      <origin xyz="0 0 0" rpy="0 0 0"/>
+      <geometry>
+        <box size="0.02 0.02 0.01"/>
+      </geometry>
+    </collision> -->
+    <visual>
+      <origin xyz="0 0 0" rpy="0 0 0"/>
+      <geometry>
+        <box size="0.02 0.02 0.01"/>
+      </geometry>
+      <material name="green"/>
+    </visual>
+    <inertial>
+      <mass value="1e-5" />
+      <origin xyz="0 0 0" rpy="0 0 0"/>
+      <inertia ixx="1e-6" ixy="0" ixz="0" iyy="1e-6" iyz="0" izz="1e-6" />
+    </inertial>
+  </link>
+  <gazebo reference="front_right_corner_camera_link">
+    <material>Gazebo/Green</material>
+  </gazebo>
+  <joint name="front_right_corner_camera_joint" type="fixed">
+    <origin xyz="0.5 -0.6535 1.75" rpy="0 0.785 -0.785"/>
+    <parent link="base_link"/>
+    <child link="front_right_corner_camera_link"/>
+    <axis xyz="0 0 0" />
+  </joint>
+  <!-- Rear Left Corner Camera -->
+  <link name="rear_left_corner_camera_link">
+    <!-- <collision>
+      <origin xyz="0 0 0" rpy="0 0 0"/>
+      <geometry>
+        <box size="0.02 0.02 0.01"/>
+      </geometry>
+    </collision> -->
+    <visual>
+      <origin xyz="0 0 0" rpy="0 0 0"/>
+      <geometry>
+        <box size="0.02 0.02 0.01"/>
+      </geometry>
+      <material name="blue"/>
+    </visual>
+    <inertial>
+      <mass value="1e-5" />
+      <origin xyz="0 0 0" rpy="0 0 0"/>
+      <inertia ixx="1e-6" ixy="0" ixz="0" iyy="1e-6" iyz="0" izz="1e-6" />
+    </inertial>
+  </link>
+  <gazebo reference="rear_left_corner_camera_link">
+    <material>Gazebo/Blue</material>
+  </gazebo>
+  <joint name="rear_left_corner_camera_joint" type="fixed">
+    <origin xyz="-1.0 0.6545 1.75" rpy="0 0.785 2.356"/>
+    <parent link="base_link"/>
+    <child link="rear_left_corner_camera_link"/>
+    <axis xyz="0 0 0" />
+  </joint>
+  <!-- Rear Right Corner Camera -->
+  <link name="rear_right_corner_camera_link">
+    <!-- <collision>
+      <origin xyz="0 0 0" rpy="0 0 0"/>
+      <geometry>
+        <box size="0.02 0.02 0.01"/>
+      </geometry>
+    </collision> -->
+    <visual>
+      <origin xyz="0 0 0" rpy="0 0 0"/>
+      <geometry>
+        <box size="0.02 0.02 0.01"/>
+      </geometry>
+      <material name="yellow"/>
+    </visual>
+    <inertial>
+      <mass value="1e-5" />
+      <origin xyz="0 0 0" rpy="0 0 0"/>
+      <inertia ixx="1e-6" ixy="0" ixz="0" iyy="1e-6" iyz="0" izz="1e-6" />
+    </inertial>
+  </link>
+  <gazebo reference="rear_right_corner_camera_link">
+    <material>Gazebo/Yellow</material>
+  </gazebo>
+  <joint name="rear_right_corner_camera_joint" type="fixed">
+    <origin xyz="-1.0 -0.6535 1.75" rpy="0 0.785 -2.356"/>
+    <parent link="base_link"/>
+    <child link="rear_right_corner_camera_link"/>
+    <axis xyz="0 0 0" />
+  </joint>
+    <!--
+  <link name="stereo_camera_link">
+    <collision>
+      <origin xyz="0 0 0" rpy="0 0 0"/>
+      <geometry>
+        <box size="0.05 0.05 0.05"/>
+      </geometry>
+    </collision>
+    <visual>
+      <origin xyz="0 0 0" rpy="0 0 0"/>
+      <geometry>
+        <box size="0.05 0.05 0.05"/>
+      </geometry>
+      <material name="red"/>
+    </visual>
+    <inertial>
+      <mass value="1e-5" />
+      <origin xyz="0 0 0" rpy="0 0 0"/>
+      <inertia ixx="1e-6" ixy="0" ixz="0" iyy="1e-6" iyz="0" izz="1e-6" />
+    </inertial>
+  </link>
+  <joint name="gem_stereo_camera_joint" type="fixed">
+    <origin xyz="-0.045 0 0" rpy="-1.5708 3.1416 0"/>
+    <parent link="front_camera_link"/>
+    <child link="stereo_camera_link"/>
+  </joint>
+  -->
+  <!-- IMU -->
+  <link name="IMU_link">
+    <collision>
+      <origin xyz="0 0 0" rpy="0 0 0"/>
+      <geometry>
+        <box size="0.1 0.1 0.1"/>
+      </geometry>
+    </collision>
+    <visual>
+      <origin xyz="0 0 0" rpy="0 0 0"/>
+      <geometry>
+        <box size="0.1 0.1 0.1"/>
+      </geometry>
+      <material name="red"/>
+    </visual>
+    <inertial>
+      <origin xyz="0 0 0" rpy="0 0 0"/>
+      <mass value="1"/>
+      <inertia
+        ixx="1.0" ixy="0.0" ixz="0.0"
+        iyy="1.0" iyz="0.0"
+        izz="1.0"/>
+    </inertial>
+  </link>
+  <gazebo reference="IMU_link">
+    <material>Gazebo/White</material>
+  </gazebo>
+  <joint name="IMU_joint" type="fixed">
+    <origin xyz="-0.246 0 0.05" rpy="0 0 -1.5708"/>
+    <parent link="base_link"/>
+    <child link="IMU_link"/>
+  </joint>
+  <!-- GPS -->
+  <link name="GPS_link">
+    <collision>
+      <origin xyz="0 0 0" rpy="0 0 0"/>
+      <geometry>
+        <box size="0.1 0.1 0.1"/>
+      </geometry>
+    </collision>
+    <visual>
+      <origin xyz="0 0 0" rpy="0 0 0"/>
+      <geometry>
+        <box size="0.1 0.1 0.1"/>
+      </geometry>
+      <material name="red"/>
+    </visual>
+    <inertial>
+      <origin xyz="0 0 0" rpy="0 0 0"/>
+      <mass value="1"/>
+      <inertia
+        ixx="1.0" ixy="0.0" ixz="0.0"
+        iyy="1.0" iyz="0.0"
+        izz="1.0"/>
+    </inertial>
+  </link>
+  <gazebo reference="GPS_link">
+    <material>Gazebo/White</material>
+  </gazebo>
+  <joint name="GPS_joint" type="fixed">
+    <origin xyz="-0.246 0 0.05" rpy="0 0 0"/>
+    <parent link="base_link"/>
+    <child link="GPS_link"/>
   </joint>
   <!-- *********************************** Front Left Wheel *********************************** -->
@@ -976,313 +1234,3 @@
   <xacro:steering_hinge_transmission name="left_steering_hinge" />
   <xacro:steering_hinge_transmission name="right_steering_hinge" />
-  <!-- *********************************************** Sensors ************************************************ -->
-  <xacro:OS1_64 parent="top_rack_link" name="os_sensor" topic_points="/ouster/points" topic_imu ="/ouster/imu" hz="10" lasers="64" samples="512" min_range="0.9" max_range="75.0" noise="0.008" min_angle="-${M_PI}" max_angle="${M_PI}" lidar_link="os_lidar" imu_link="os_imu" vfov_min="-.26" vfov_max=".26" >
-    <origin xyz="0.02 0.42 0" rpy="1.5708 0 3.1416" />
-  </xacro:OS1_64>
-  <!-- ************************* Front Camera ************************* -->
-  <link name="front_single_camera_link">
-    <collision>
-      <origin xyz="0 0 0" rpy="0 0 0"/>
-      <geometry>
-        <box size="0.05 0.05 0.05"/>
-      </geometry>
-    </collision>
-    <visual>
-      <origin xyz="0 0 0" rpy="0 0 0"/>
-      <geometry>
-        <box size="0.05 0.05 0.05"/>
-      </geometry>
-      <material name="red"/>
-    </visual>
-    <inertial>
-      <mass value="1e-5" />
-      <origin xyz="0 0 0" rpy="0 0 0"/>
-      <inertia ixx="1e-6" ixy="0" ixz="0" iyy="1e-6" iyz="0" izz="1e-6" />
-    </inertial>
-  </link>
-  <gazebo reference="front_single_camera_link">
-    <material>Gazebo/White</material>
-  </gazebo>
-  <!--
-  <joint name="gem_front_camera_joint" type="fixed">
-    <origin xyz="-0.045 0 0" rpy="-1.5708 3.1416 0"/>
-    <parent link="front_camera_link"/>
-    <child link="front_single_camera_link"/>
-  </joint>
-  -->
-  <joint name="gem_front_camera_joint" type="fixed">
-    <origin xyz="0 0 0" rpy="0 -1.57 0"/>
-    <parent link="front_camera_link"/>
-    <child link="front_single_camera_link"/>
-  </joint>
-  <!-- ************************* Corner Cameras ************************* -->
-  <!-- Front Left Corner Camera -->
-  <link name="front_left_corner_camera_link">
-    <!-- <collision>
-      <origin xyz="0 0 0" rpy="0 0 0"/>
-      <geometry>
-        <box size="0.02 0.02 0.01"/>
-      </geometry>
-    </collision> -->
-    <visual>
-      <origin xyz="0 0 0" rpy="0 0 0"/>
-      <geometry>
-        <box size="0.02 0.02 0.01"/>
-      </geometry>
-      <material name="red"/>
-    </visual>
-    <inertial>
-      <mass value="1e-5" />
-      <origin xyz="0 0 0" rpy="0 0 0"/>
-      <inertia ixx="1e-6" ixy="0" ixz="0" iyy="1e-6" iyz="0" izz="1e-6" />
-    </inertial>
-  </link>
-  <gazebo reference="front_left_corner_camera_link">
-    <material>Gazebo/Red</material>
-  </gazebo>
-  <joint name="front_left_corner_camera_joint" type="fixed">
-    <origin xyz="0.5 0.6545 1.75" rpy="0 0.785 0.785"/>
-    <parent link="base_link"/>
-    <child link="front_left_corner_camera_link"/>
-    <axis xyz="0 0 0" />
-  </joint>
-  <!-- Front Right Corner Camera -->
-  <link name="front_right_corner_camera_link">
-    <!-- <collision>
-      <origin xyz="0 0 0" rpy="0 0 0"/>
-      <geometry>
-        <box size="0.02 0.02 0.01"/>
-      </geometry>
-    </collision> -->
-    <visual>
-      <origin xyz="0 0 0" rpy="0 0 0"/>
-      <geometry>
-        <box size="0.02 0.02 0.01"/>
-      </geometry>
-      <material name="green"/>
-    </visual>
-    <inertial>
-      <mass value="1e-5" />
-      <origin xyz="0 0 0" rpy="0 0 0"/>
-      <inertia ixx="1e-6" ixy="0" ixz="0" iyy="1e-6" iyz="0" izz="1e-6" />
-    </inertial>
-  </link>
-  <gazebo reference="front_right_corner_camera_link">
-    <material>Gazebo/Green</material>
-  </gazebo>
-  <joint name="front_right_corner_camera_joint" type="fixed">
-    <origin xyz="0.5 -0.6535 1.75" rpy="0 0.785 -0.785"/>
-    <parent link="base_link"/>
-    <child link="front_right_corner_camera_link"/>
-    <axis xyz="0 0 0" />
-  </joint>
-  <!-- Rear Left Corner Camera -->
-  <link name="rear_left_corner_camera_link">
-    <!-- <collision>
-      <origin xyz="0 0 0" rpy="0 0 0"/>
-      <geometry>
-        <box size="0.02 0.02 0.01"/>
-      </geometry>
-    </collision> -->
-    <visual>
-      <origin xyz="0 0 0" rpy="0 0 0"/>
-      <geometry>
-        <box size="0.02 0.02 0.01"/>
-      </geometry>
-      <material name="blue"/>
-    </visual>
-    <inertial>
-      <mass value="1e-5" />
-      <origin xyz="0 0 0" rpy="0 0 0"/>
-      <inertia ixx="1e-6" ixy="0" ixz="0" iyy="1e-6" iyz="0" izz="1e-6" />
-    </inertial>
-  </link>
-  <gazebo reference="rear_left_corner_camera_link">
-    <material>Gazebo/Blue</material>
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
Commit message: update urdf for oak and livox

File: src/vehicle_drivers/gem_description/urdf/e4/gem_e4.urdf.xacro (robot description, xacro)
@@ -648,14 +648,14 @@
     <axis xyz="0 0 1" />
   </joint>
-  <link name="top_lidar_link">
-    <inertial>
-      <origin xyz="0 0 0" rpy="0 0 0" />
-      <mass value="0" />
-      <inertia ixx="0" ixy="0" ixz="0" iyy="0" iyz="0" izz="0" />
-    </inertial>
-    <visual>
-      <origin xyz="0 0 0" rpy="0 0 0" />
-      <geometry>
-        <mesh filename="package://gem_description/meshes/e4/top_lidar_link.STL" />
+  <link name="front_camera_link">
+    <inertial>
+      <origin xyz="0 0 0" rpy="0 0 0" />
+      <mass value="0" />
+      <inertia ixx="0" ixy="0" ixz="0" iyy="0" iyz="0" izz="0" />
+    </inertial>
+    <visual>
+      <origin xyz="0 0 0" rpy="0 0 0" />
+      <geometry>
+        <mesh filename="package://gem_description/meshes/e4/front_camera_link.STL" />
       </geometry>
       <material name="">
@@ -666,28 +666,28 @@
       <origin xyz="0 0 0" rpy="0 0 0" />
       <geometry>
-        <mesh filename="package://gem_description/meshes/e4/top_lidar_link.STL" />
-      </geometry>
-    </collision>
-  </link>
-  <gazebo reference="top_lidar_link">
-    <material>Gazebo/White</material>
-  </gazebo>
-  <joint name="top_lidar_joint" type="fixed">
-    <origin xyz="-0.15144 0 2.08" rpy="0 0 0" />
-    <parent link="base_link" />
-    <child link="top_lidar_link" />
-    <axis xyz="0 0 0" />
-  </joint>
-  <link name="front_camera_link">
-    <inertial>
-      <origin xyz="0 0 0" rpy="0 0 0" />
-      <mass value="0" />
-      <inertia ixx="0" ixy="0" ixz="0" iyy="0" iyz="0" izz="0" />
-    </inertial>
-    <visual>
-      <origin xyz="0 0 0" rpy="0 0 0" />
-      <geometry>
         <mesh filename="package://gem_description/meshes/e4/front_camera_link.STL" />
       </geometry>
+    </collision>
+  </link>
+  <gazebo reference="front_camera_link">
+    <material>Gazebo/White</material>
+  </gazebo>
+  <joint name="front_camera_joint" type="fixed">
+    <origin xyz="0.535 0 1.683" rpy="0 0 0" />
+    <parent link="base_link" />
+    <child link="front_camera_link" />
+    <axis xyz="0 0 0" />
+  </joint>
+  <link name="front_lidar_link">
+    <inertial>
+      <origin xyz="0 0 0" rpy="0 0 0" />
+      <mass value="0" />
+      <inertia ixx="0" ixy="0" ixz="0" iyy="0" iyz="0" izz="0" />
+    </inertial>
+    <visual>
+      <origin xyz="0 0 0" rpy="0 0 0" />
+      <geometry>
+        <mesh filename="package://gem_description/meshes/e4/front_lidar_link.STL" />
+      </geometry>
       <material name="">
         <color rgba="0.8 0.8 0.9 1" />
@@ -697,72 +697,6 @@
       <origin xyz="0 0 0" rpy="0 0 0" />
       <geometry>
-        <mesh filename="package://gem_description/meshes/e4/front_camera_link.STL" />
-      </geometry>
-    </collision>
-  </link>
-  <gazebo reference="front_camera_link">
-    <material>Gazebo/White</material>
-  </gazebo>
-  <joint name="front_camera_joint" type="fixed">
-    <origin xyz="0.535 0 1.683" rpy="0 1.5708 0" />
-    <parent link="base_link" />
-    <child link="front_camera_link" />
-    <axis xyz="0 0 0" />
-  </joint>
-  <link name="front_single_camera_link">
-    <collision>
-      <origin xyz="0 0 0" rpy="0 0 0"/>
-      <geometry>
-        <box size="0.05 0.05 0.05"/>
-      </geometry>
-    </collision>
-    <visual>
-      <origin xyz="0 0 0" rpy="0 0 0"/>
-      <geometry>
-        <box size="0.05 0.05 0.05"/>
-      </geometry>
-      <material name="red"/>
-    </visual>
-    <inertial>
-      <mass value="1e-5" />
-      <origin xyz="0 0 0" rpy="0 0 0"/>
-      <inertia ixx="1e-6" ixy="0" ixz="0" iyy="1e-6" iyz="0" izz="1e-6" />
-    </inertial>
-  </link>
-  <gazebo reference="front_single_camera_link">
-    <material>Gazebo/White</material>
-  </gazebo>
-  <!--
-  <joint name="gem_front_camera_joint" type="fixed">
-    <origin xyz="-0.045 0 0" rpy="-1.5708 3.1416 0"/>
-    <parent link="front_camera_link"/>
-    <child link="front_single_camera_link"/>
-  </joint>
-  -->
-  <joint name="gem_front_camera_joint" type="fixed">
-    <origin xyz="0 0 0" rpy="0 -1.57 0"/>
-    <parent link="front_camera_link"/>
-    <child link="front_single_camera_link"/>
-  </joint>
-  <link name="front_lidar_link">
-    <inertial>
-      <origin xyz="0 0 0" rpy="0 0 0" />
-      <mass value="0" />
-      <inertia ixx="0" ixy="0" ixz="0" iyy="0" iyz="0" izz="0" />
-    </inertial>
-    <visual>
-      <origin xyz="0 0 0" rpy="0 0 0" />
-      <geometry>
         <mesh filename="package://gem_description/meshes/e4/front_lidar_link.STL" />
       </geometry>
-      <material name="">
-        <color rgba="0.8 0.8 0.9 1" />
-      </material>
-    </visual>
-    <collision>
-      <origin xyz="0 0 0" rpy="0 0 0" />
-      <geometry>
-        <mesh filename="package://gem_description/meshes/e4/front_lidar_link.STL" />
-      </geometry>
     </collision>
   </link>
@@ -771,5 +705,5 @@
   </gazebo>
   <joint name="front_lidar_joint" type="fixed">
-    <origin xyz="0.38206 0 1.71" rpy="0 0 0" />
+    <origin xyz="0.38206 0 1.71" rpy="0 0.3 0" />
     <parent link="base_link" />
     <child link="front_lidar_link" />
@@ -913,4 +847,12 @@
     <axis xyz="0 0 0" />
   </joint>
+    <!-- Front Right Corner Camera Optical Frame (For ROS Image/CameraInfo messages) -->
+  <link name="front_right_corner_camera_optical_frame"/>
+  <joint name="front_right_corner_camera_optical_joint" type="fixed">
+    <!-- -90 deg Roll, -90 deg Yaw rotation to align body frame with optical frame -->
+    <origin xyz="0 0 0" rpy="-1.5707963 0 -1.5707963"/>
+    <parent link="front_right_corner_camera_link"/>
+    <child link="front_right_corner_camera_optical_frame"/>
+  </joint>
   <!-- Rear Left Corner Camera -->
   <link name="rear_left_corner_camera_link">
@@ -943,4 +885,12 @@
     <axis xyz="0 0 0" />
   </joint>
+  <!-- Rear Left Corner Camera Optical Frame (For ROS Image/CameraInfo messages) -->
+  <link name="rear_left_corner_camera_optical_frame"/>
+  <joint name="rear_left_corner_camera_optical_joint" type="fixed">
+    <!-- -90 deg Roll, -90 deg Yaw rotation to align body frame with optical frame -->
+    <origin xyz="0 0 0" rpy="-1.5707963 0 -1.5707963"/>
+    <parent link="rear_left_corner_camera_link"/>
+    <child link="rear_left_corner_camera_optical_frame"/>
+  </joint>
   <!-- Rear Right Corner Camera -->
   <link name="rear_right_corner_camera_link">
@@ -973,31 +923,12 @@
     <axis xyz="0 0 0" />
   </joint>
-    <!--
-  <link name="stereo_camera_link">
-    <collision>
-      <origin xyz="0 0 0" rpy="0 0 0"/>
-      <geometry>
-        <box size="0.05 0.05 0.05"/>
-      </geometry>
-    </collision>
-    <visual>
-      <origin xyz="0 0 0" rpy="0 0 0"/>
-      <geometry>
-        <box size="0.05 0.05 0.05"/>
-      </geometry>
-      <material name="red"/>
-    </visual>
-    <inertial>
-      <mass value="1e-5" />
-      <origin xyz="0 0 0" rpy="0 0 0"/>
-      <inertia ixx="1e-6" ixy="0" ixz="0" iyy="1e-6" iyz="0" izz="1e-6" />
-    </inertial>
-  </link>
-  <joint name="gem_stereo_camera_joint" type="fixed">
-    <origin xyz="-0.045 0 0" rpy="-1.5708 3.1416 0"/>
-    <parent link="front_camera_link"/>
-    <child link="stereo_camera_link"/>
-  </joint>
-  -->
+  <!-- Rear Right Corner Camera Optical Frame (For ROS Image/CameraInfo messages) -->
+  <link name="rear_right_corner_camera_optical_frame"/>
+  <joint name="rear_right_corner_camera_optical_joint" type="fixed">
+    <!-- -90 deg Roll, -90 deg Yaw rotation to align body frame with optical frame -->
+    <origin xyz="0 0 0" rpy="-1.5707963 0 -1.5707963"/>
+    <parent link="rear_right_corner_camera_link"/>
+    <child link="rear_right_corner_camera_optical_frame"/>
+  </joint>
   <!-- IMU -->
   <link name="IMU_link">
