Commit message: code refactoring

File: src/vehicle_drivers/gem_description/urdf/e2/gem_e2.urdf.xacro (robot description, xacro)
@@ -12,49 +12,39 @@
   <xacro:include filename="$(find gem_description)/urdf/ouster/OS1-64.urdf.xacro" />
   <!-- *************************** Base link below *************************** -->
+  <!-- Main structural frame of the vehicle -->
+  <link name="base_link">
+    <inertial>
+      <origin xyz="0 0 0" rpy="0 0 0" />
+      <mass value="686" />
+      <inertia
+        ixx="325"
+        ixy="0"
+        ixz="0"
+        iyy="597"
+        iyz="0"
+        izz="465" />
+    </inertial>
+    <visual>
+      <origin xyz="0 0 0" rpy="0 0 0" />
+      <geometry>
+        <mesh filename="package://gem_description/meshes/e2/base_link.STL" />
+      </geometry>
+      <material name="white" />
+    </visual>
+    <collision>
+      <origin xyz="0 0 0" rpy="0 0 0" />
+      <geometry>
+        <mesh filename="package://gem_description/meshes/e2/base_link.STL" />
+      </geometry>
+    </collision>
+  </link>
+  <!-- Ground projection link (2D level ground frame) -->
   <link name="base_footprint">
   </link>
-  <link name="base_link">
-    <!--
-    <inertial>
-      <origin xyz="0.0410109641324594 0.000349767124208047 0.219524161679779" rpy="0 0 0" />
-      <mass value="686.066668067387" />
-      <inertia
-        ixx="205.702789313137"
-        ixy="-0.20742120719075"
-        ixz="-9.13771633467953"
-        iyy="482.020173559149"
-        iyz="0.0517191981605489"
-        izz="482.316418870047" />
-    </inertial>
-    -->
-    <inertial>
-      <origin xyz="0 0 0" rpy="0 0 0" />
-      <mass value="686" />
-      <inertia
-        ixx="325"
-        ixy="0"
-        ixz="0"
-        iyy="597"
-        iyz="0"
-        izz="465" />
-    </inertial>
-    <visual>
-      <origin xyz="0 0 0" rpy="0 0 0" />
-      <geometry>
-        <mesh filename="package://gem_description/meshes/e2/base_link.STL" />
-      </geometry>
-      <material name="white" />
-    </visual>
-    <collision>
-      <origin xyz="0 0 0" rpy="0 0 0" />
-      <geometry>
-        <mesh filename="package://gem_description/meshes/e2/base_link.STL" />
-      </geometry>
-    </collision>
-  </link>
-  <joint name="base_link" type="fixed">
-    <origin xyz="0 0 0.44" rpy="0 0 0"/>
-    <parent link="base_footprint"/>
-    <child link="base_link"/>
+  <!-- Joint directing base_link -> base_footprint (-0.44m down to the ground) -->
+  <joint name="base_footprint_joint" type="fixed">
+    <origin xyz="0 0 -0.44" rpy="0 0 0"/>
+    <parent link="base_link"/>
+    <child link="base_footprint"/>
   </joint>
   <!-- ******************************************* Fixed links below ******************************************* -->

File: src/vehicle_drivers/gem_description/urdf/e4/gem_e4.urdf.xacro (robot description, xacro)
@@ -13,6 +13,4 @@
   <xacro:include filename="$(find gem_description)/urdf/macros.xacro" />
   <xacro:include filename="$(find gem_description)/urdf/ouster/OS1-64.urdf.xacro" />
-  <link name="base_footprint">
-  </link>
   <link name="base_link">
     <inertial>
@@ -46,8 +44,10 @@
     <material>Gazebo/Blue</material>
   </gazebo>
-  <joint name="base_link" type="fixed">
-    <origin xyz="0 0 0.268" rpy="0 0 0" />
-    <parent link="base_footprint" />
-    <child link="base_link" />
+  <link name="base_footprint">
+  </link>
+  <joint name="base_footprint_joint" type="fixed">
+    <origin xyz="0 0 -0.268" rpy="0 0 0" />
+    <parent link="base_link" />
+    <child link="base_footprint" />
   </joint>
   <!-- ************************************* Fixed Links ************************************* -->

Commit message: add e2 corner cameras link, livox lidar, zed and oak camera mount links

File: src/vehicle_drivers/gem_description/urdf/e2/gem_e2.urdf.xacro (robot description, xacro)
@@ -1012,8 +1012,8 @@
   <!-- *********************************************** Sensors ************************************************ -->
  <xacro:OS1_64 parent="top_rack_link" name="os_sensor" topic_points="/ouster/points" topic_imu ="/ouster/imu" hz="10" lasers="64" samples="512" min_range="0.9" max_range="75.0" noise="0.008" min_angle="-${M_PI}" max_angle="${M_PI}" lidar_link="os_lidar" imu_link="os_imu" vfov_min="-.26" vfov_max=".26" >
-    <origin xyz="0.02 0.115 -0.6575" rpy="1.5708 0 3.1416" />
+    <origin xyz="0.02 0.115 -0.6575" rpy="-1.5708 0 0" />
   </xacro:OS1_64>
-  <!-- ************************* Front Camera ************************* -->
-  <link name="front_single_camera_link">
+  <!-- ************************* Front Zed Camera ************************* -->
+  <link name="zed_camera_link">
     <collision>
       <origin xyz="0 0 0" rpy="0 0 0"/>
@@ -1035,43 +1035,9 @@
     </inertial>
   </link>
-  <!--
-  <joint name="gem_front_camera_joint" type="fixed">
-    <origin xyz="-0.045 0 0" rpy="-1.5708 3.1416 0"/>
-    <parent link="front_camera_link"/>
-    <child link="front_single_camera_link"/>
-  </joint>
-  -->
-  <joint name="gem_front_camera_joint" type="fixed">
-    <origin xyz="0.394 0 1.19" rpy="0 0 0"/>
+  <joint name="zed_camera_joint" type="fixed">
+    <origin xyz="0.394 0 1.35" rpy="0 0 0"/>
     <parent link="base_link"/>
-    <child link="front_single_camera_link"/>
-  </joint>
-  <!--
-  <link name="stereo_camera_link">
-    <collision>
-      <origin xyz="0 0 0" rpy="0 0 0"/>
-      <geometry>
-        <box size="0.05 0.05 0.05"/>
-      </geometry>
-    </collision>
-    <visual>
-      <origin xyz="0 0 0" rpy="0 0 0"/>
-      <geometry>
-        <box size="0.05 0.05 0.05"/>
-      </geometry>
-      <material name="red"/>
-    </visual>
-    <inertial>
-      <mass value="1e-5" />
-      <origin xyz="0 0 0" rpy="0 0 0"/>
-      <inertia ixx="1e-6" ixy="0" ixz="0" iyy="1e-6" iyz="0" izz="1e-6" />
-    </inertial>
-  </link>
-  <joint name="gem_stereo_camera_joint" type="fixed">
-    <origin xyz="-0.045 0 0" rpy="-1.5708 3.1416 0"/>
-    <parent link="front_camera_link"/>
-    <child link="stereo_camera_link"/>
-  </joint>
-  -->
+    <child link="zed_camera_link"/>
+  </joint>
   <!-- IMU -->
   <link name="IMU_link">
@@ -1138,55 +1104,80 @@
     <child link="GPS_link"/>
   </joint>
-  <!-- Front Sonar -->
-  <link name="front_sonar_link">
-    <inertial>
-      <mass value="0.001" />
-      <origin xyz="0 0 0" rpy="0 0 0" />
-      <inertia ixx="0.000000017" ixy="0" ixz="0" iyy="0.000000017" iyz="0" izz="0.000000017" />
-    </inertial>
-    <visual>
-      <origin xyz="0 0 0" rpy="0 0 0" />
-      <geometry>
-        <box size="0.05 0.2 0.1" />
-      </geometry>
-    <material name="orange"/>
-    </visual>
-    <collision>
-      <origin xyz="0 0 0" rpy="0 0 0" />
-      <geometry>
-        <box size="0.05 0.2 0.1" />
-      </geometry>
-    </collision>
-  </link>
-  <joint name="front_sonar_joint" type="fixed">
-    <origin xyz="0 0.38 0.065" rpy="0 -1.5708 -1.5708"/>
-    <parent link="front_rack_link"/>
-    <child link="front_sonar_link"/>
-  </joint>
-  <!-- Rear Sonar -->
-  <link name="rear_sonar_link">
-    <inertial>
-      <mass value="0.001" />
-      <origin xyz="0 0 0" rpy="0 0 0" />
-      <inertia ixx="0.000000017" ixy="0" ixz="0" iyy="0.000000017" iyz="0" izz="0.000000017" />
-    </inertial>
-    <visual>
-      <origin xyz="0 0 0" rpy="0 0 0" />
-      <geometry>
-        <box size="0.05 0.2 0.1" />
-      </geometry>
-    <material name="orange"/>
-    </visual>
-    <collision>
-      <origin xyz="0 0 0" rpy="0 0 0" />
-      <geometry>
-        <box size="0.05 0.2 0.1" />
-      </geometry>
-    </collision>
-  </link>
-  <joint name="rear_sonar_joint" type="fixed">
-    <origin xyz="0 0.38 0.065" rpy="0 -1.5708 -1.5708"/>
-    <parent link="rear_rack_link"/>
-    <child link="rear_sonar_link"/>
+   <!-- ************************* Corner Cameras ************************* -->
+  <!-- Front Left Corner Camera -->
+  <link name="front_left_corner_camera_link">
+    <!-- <collision>
+      <origin xyz="0 0 0" rpy="0 0 0"/>
+      <geometry>
+        <box size="0.02 0.02 0.01"/>
+      </geometry>
+    </collision> -->
+    <visual>
+      <origin xyz="0 0 0" rpy="0 0 0"/>
+      <geometry>
+        <box size="0.02 0.02 0.01"/>
+      </geometry>
+      <material name="red"/>
+    </visual>
+    <inertial>
+      <mass value="1e-5" />
+      <origin xyz="0 0 0" rpy="0 0 0"/>
+      <inertia ixx="1e-6" ixy="0" ixz="0" iyy="1e-6" iyz="0" izz="1e-6" />
+    </inertial>
+  </link>
+  <gazebo reference="front_left_corner_camera_link">
+    <material>Gazebo/Red</material>
+  </gazebo>
+  <joint name="front_left_corner_camera_joint" type="fixed">
+    <origin xyz="0.1 0.6545 1.45" rpy="0 0.785 0.785"/>
+    <parent link="base_link"/>
+    <child link="front_left_corner_camera_link"/>
+    <axis xyz="0 0 0" />
+  </joint>
+  <!-- Front Left Corner Camera Optical Frame (For ROS Image/CameraInfo messages) -->
+  <link name="front_left_corner_camera_optical_frame"/>
+  <joint name="front_left_corner_camera_optical_joint" type="fixed">
+    <!-- -90 deg Roll, -90 deg Yaw rotation to align body frame with optical frame -->
+    <origin xyz="0 0 0" rpy="-1.5707963 0 -1.5707963"/>
+    <parent link="front_left_corner_camera_link"/>
+    <child link="front_left_corner_camera_optical_frame"/>
+  </joint>
+  <!-- Front Right Corner Camera -->
+  <link name="front_right_corner_camera_link">
+    <!-- <collision>
+      <origin xyz="0 0 0" rpy="0 0 0"/>
+      <geometry>
+        <box size="0.02 0.02 0.01"/>
+      </geometry>
+    </collision> -->
+    <visual>
+      <origin xyz="0 0 0" rpy="0 0 0"/>
+      <geometry>
+        <box size="0.02 0.02 0.01"/>
+      </geometry>
+      <material name="green"/>
+    </visual>
+    <inertial>
+      <mass value="1e-5" />
+      <origin xyz="0 0 0" rpy="0 0 0"/>
+      <inertia ixx="1e-6" ixy="0" ixz="0" iyy="1e-6" iyz="0" izz="1e-6" />
+    </inertial>
+  </link>
+  <gazebo reference="front_right_corner_camera_link">
+    <material>Gazebo/Green</material>
+  </gazebo>
+  <joint name="front_right_corner_camera_joint" type="fixed">
+    <origin xyz="0.1 -0.6535 1.45" rpy="0 0.785 -0.785"/>
+    <parent link="base_link"/>
+    <child link="front_right_corner_camera_link"/>
+    <axis xyz="0 0 0" />
+  </joint>
+    <!-- Front Right Corner Camera Optical Frame (For ROS Image/CameraInfo messages) -->
+  <link name="front_right_corner_camera_optical_frame"/>
+  <joint name="front_right_corner_camera_optical_joint" type="fixed">
+    <!-- -90 deg Roll, -90 deg Yaw rotation to align body frame with optical frame -->
+    <origin xyz="0 0 0" rpy="-1.5707963 0 -1.5707963"/>
+    <parent link="front_right_corner_camera_link"/>
+    <child link="front_right_corner_camera_optical_frame"/>
   </joint>
 </robot>

File: src/vehicle_drivers/gem_description/urdf/e4/gem_e4.urdf.xacro (robot description, xacro)
@@ -648,14 +648,45 @@
     <axis xyz="0 0 1" />
   </joint>
-  <link name="front_camera_link">
-    <inertial>
-      <origin xyz="0 0 0" rpy="0 0 0" />
-      <mass value="0" />
-      <inertia ixx="0" ixy="0" ixz="0" iyy="0" iyz="0" izz="0" />
-    </inertial>
-    <visual>
-      <origin xyz="0 0 0" rpy="0 0 0" />
-      <geometry>
-        <mesh filename="package://gem_description/meshes/e4/front_camera_link.STL" />
+  <!-- ************************* Front Oak Camera ************************* -->
+  <link name="oak_link">
+    <inertial>
+      <origin xyz="0 0 0" rpy="0 0 0" />
+      <mass value="0" />
+      <inertia ixx="0" ixy="0" ixz="0" iyy="0" iyz="0" izz="0" />
+    </inertial>
+    <visual>
+      <origin xyz="0 0 0" rpy="1.57 0 -1.57" />
+      <geometry>
+        <mesh filename="package://gem_description/meshes/e4/OAK-D-LR.stl" />
+      </geometry>
+      <material name="white"/>
+    </visual>
+    <collision>
+      <origin xyz="0 0 0" rpy="0 0 0" />
+      <geometry>
+        <mesh filename="package://gem_description/meshes/e4/OAK-D-LR.stl" />
+      </geometry>
+    </collision>
+  </link>
+  <gazebo reference="oak_link">
+    <material>Gazebo/White</material>
+  </gazebo>
+  <joint name="oak_joint" type="fixed">
+    <origin xyz="0.535 0 1.683" rpy="0 0 0" />
+    <parent link="base_link" />
+    <child link="oak_link" />
+    <axis xyz="0 0 0" />
+  </joint>
+  <!-- ************************* Front Livox Lidar ************************* -->
+  <link name="livox_lidar_link">
+    <inertial>
+      <origin xyz="0 0 0" rpy="0 0 0" />
+      <mass value="0" />
+      <inertia ixx="0" ixy="0" ixz="0" iyy="0" iyz="0" izz="0" />
+    </inertial>
+    <visual>
+      <origin xyz="0 0 0" rpy="0 0 0" />
+      <geometry>
+        <mesh filename="package://gem_description/meshes/e4/livox_lidar.STL" />
       </geometry>
       <material name="">
@@ -666,46 +697,15 @@
       <origin xyz="0 0 0" rpy="0 0 0" />
       <geometry>
-        <mesh filename="package://gem_description/meshes/e4/front_camera_link.STL" />
-      </geometry>
-    </collision>
-  </link>
-  <gazebo reference="front_camera_link">
-    <material>Gazebo/White</material>
-  </gazebo>
-  <joint name="front_camera_joint" type="fixed">
-    <origin xyz="0.535 0 1.683" rpy="0 0 0" />
-    <parent link="base_link" />
-    <child link="front_camera_link" />
-    <axis xyz="0 0 0" />
-  </joint>
-  <link name="front_lidar_link">
-    <inertial>
-      <origin xyz="0 0 0" rpy="0 0 0" />
-      <mass value="0" />
-      <inertia ixx="0" ixy="0" ixz="0" iyy="0" iyz="0" izz="0" />
-    </inertial>
-    <visual>
-      <origin xyz="0 0 0" rpy="0 0 0" />
-      <geometry>
-        <mesh filename="package://gem_description/meshes/e4/front_lidar_link.STL" />
-      </geometry>
-      <material name="">
-        <color rgba="0.8 0.8 0.9 1" />
-      </material>
-    </visual>
-    <collision>
-      <origin xyz="0 0 0" rpy="0 0 0" />
-      <geometry>
-        <mesh filename="package://gem_description/meshes/e4/front_lidar_link.STL" />
-      </geometry>
-    </collision>
-  </link>
-  <gazebo reference="front_lidar_link">
-    <material>Gazebo/White</material>
-  </gazebo>
-  <joint name="front_lidar_joint" type="fixed">
-    <origin xyz="0.38206 0 1.71" rpy="0 0.3 0" />
-    <parent link="base_link" />
-    <child link="front_lidar_link" />
+        <mesh filename="package://gem_description/meshes/e4/livox_lidar.STL" />
+      </geometry>
+    </collision>
+  </link>
+  <gazebo reference="livox_lidar_link">
+    <material>Gazebo/White</material>
+  </gazebo>
+  <joint name="livox_lidar_joint" type="fixed">
+    <origin xyz="0.4 0 1.78" rpy="0 0.323 0.018" />
+    <parent link="base_link" />
+    <child link="livox_lidar_link" />
     <axis xyz="0 0 0" />
   </joint>

Commit message: add troubleshooting doc, fix imu link on e4

File: src/vehicle_drivers/gem_description/urdf/e2/gem_e2.urdf.xacro (robot description, xacro)
@@ -1041,5 +1041,5 @@
   </joint>
   <!-- IMU -->
-  <link name="IMU_link">
+  <link name="imu_link">
     <collision>
       <origin xyz="0 0 0" rpy="0 0 0"/>
@@ -1064,13 +1064,13 @@
     </inertial>
   </link>
-  <joint name="IMU_joint" type="fixed">
+  <joint name="imu_joint" type="fixed">
     <origin xyz="-0.05 -0.4 0.05" rpy="0 0 0"/>
     <parent link="base_link"/>
-    <child link="IMU_link"/>
+    <child link="imu_link"/>
   </joint>
   <link name="vsm"/>
   <joint name="velocity_sensor_joint" type="fixed">
     <origin xyz="0.0 0 0.0" rpy="0 0 0"/>
-    <parent link="IMU_link"/>
+    <parent link="imu_link"/>
     <child link="vsm"/>
   </joint>

File: src/vehicle_drivers/gem_description/urdf/e4/gem_e4.urdf.xacro (robot description, xacro)
@@ -656,5 +656,5 @@
     </inertial>
     <visual>
-      <origin xyz="0 0 0" rpy="1.57 0 -1.57" />
+      <origin xyz="0 0 0" rpy="1.57 0 1.57" />
       <geometry>
         <mesh filename="package://gem_description/meshes/e4/OAK-D-LR.stl" />
@@ -930,36 +930,4 @@
     <parent link="rear_right_corner_camera_link"/>
     <child link="rear_right_corner_camera_optical_frame"/>
-  </joint>
-  <!-- IMU -->
-  <link name="IMU_link">
-    <collision>
-      <origin xyz="0 0 0" rpy="0 0 0"/>
-      <geometry>
-        <box size="0.1 0.1 0.1"/>
-      </geometry>
-    </collision>
-    <visual>
-      <origin xyz="0 0 0" rpy="0 0 0"/>
-      <geometry>
-        <box size="0.1 0.1 0.1"/>
-      </geometry>
-      <material name="red"/>
-    </visual>
-    <inertial>
-      <origin xyz="0 0 0" rpy="0 0 0"/>
-      <mass value="1"/>
-      <inertia
-        ixx="1.0" ixy="0.0" ixz="0.0"
-        iyy="1.0" iyz="0.0"
-        izz="1.0"/>
-    </inertial>
-  </link>
-  <gazebo reference="IMU_link">
-    <material>Gazebo/White</material>
-  </gazebo>
-  <joint name="IMU_joint" type="fixed">
-    <origin xyz="-0.246 0 0.05" rpy="0 0 -1.5708"/>
-    <parent link="base_link"/>
-    <child link="IMU_link"/>
   </joint>
   <!-- GPS -->
